Commit message: Implement the IMU sensor and gimbal controller

File: metav_description/urdf/common/omni_wheel.xacro (robot description, xacro)
@@ -19,4 +19,7 @@
                               scale="0.001 0.001 0.001"/>
                     </geometry>
+                    <material name="black">
+                        <color rgba="0.000 0.000 0.000 1.000"/>
+                    </material>
                 </visual>
                 <collision>
@@ -51,5 +54,4 @@
             <kp value="1000000.0"/>
             <kd value="100.0"/>
-            <material>Gazebo/Black</material>
         </gazebo>
     </xacro:macro>
@@ -112,18 +114,19 @@
     </xacro:macro>
     <xacro:macro name="wheel_transmission" params="prefix mechanical_reduction">
-            <transmission name="${prefix}_wheel_trans">
-                <plugin>transmission_interface/SimpleTransmission</plugin>
-                <actuator name="${prefix}_wheel_motor" role="${prefix}_wheel_motor"/>
-                <joint name="${prefix}_wheel_joint" role="${prefix}_wheel_joint">
-                    <mechanical_reduction>${mechanical_reduction}</mechanical_reduction>
-                    <offset>0.0</offset>
-                </joint>
-            </transmission>
-            <joint name="${prefix}_wheel_joint">
-                <command_interface name="velocity">
-                </command_interface>
-                <state_interface name="position"/>
-                <state_interface name="velocity"/>
+        <transmission name="${prefix}_wheel_trans">
+            <plugin>transmission_interface/SimpleTransmission</plugin>
+            <actuator name="${prefix}_wheel_motor" role="${prefix}_wheel_motor"/>
+            <joint name="${prefix}_wheel_joint" role="${prefix}_wheel_joint">
+                <mechanical_reduction>${mechanical_reduction}</mechanical_reduction>
+                <offset>0.0</offset>
             </joint>
+        </transmission>
+        <joint name="${prefix}_wheel_joint">
+            <command_interface name="effort">
+            </command_interface>
+            <state_interface name="position"/>
+            <state_interface name="velocity"/>
+            <state_interface name="effort"/>
+        </joint>
     </xacro:macro>
 </robot>

File: metav_description/urdf/sentry/sentry.gazebo.xacro (robot description, xacro)
@@ -18,6 +18,6 @@
             <publish_nested_model_pose>true</publish_nested_model_pose>
             <use_pose_vector_msg>true</use_pose_vector_msg>
-            <!-- <static_publisher>true</static_publisher>
-            <static_update_frequency>-1</static_update_frequency> -->
+            <static_publisher>true</static_publisher>
+            <static_update_frequency>-1</static_update_frequency>
         </plugin>
     </gazebo>

File: metav_description/urdf/sentry/sentry.xacro (robot description, xacro)
@@ -13,4 +13,8 @@
     <xacro:include filename="$(find metav_description)/urdf/sentry/sentry.chassis.xacro"/>
     <xacro:chassis roller_type="$(arg roller_type)"/>
+    <xacro:include filename="$(find metav_description)/urdf/sentry/sentry.gimbal.xacro"/>
+    <xacro:gimbal/>
+    <xacro:include filename="$(find metav_description)/urdf/common/sensor_imu.xacro"/>
+    <xacro:sensor_imu connected_to="pitch_gimbal" imu_name="gimbal_imu" xyz="0 0 0.1"/>
     <ros2_control name="sentry_control" type="system">
         <xacro:if value="$(arg is_simulation)">
@@ -23,4 +27,6 @@
         <xacro:wheel_transmission prefix="left" mechanical_reduction="20.0"/>
         <xacro:wheel_transmission prefix="back" mechanical_reduction="20.0"/>
+        <xacro:gimbal_transmission prefix="yaw" mechanical_reduction="1.0"/>
+        <xacro:gimbal_transmission prefix="pitch" mechanical_reduction="1.0"/>
     </ros2_control>
     <xacro:if value="$(arg is_simulation)">
