Commit message: Fix all yaw gimbal related problems in real hardware

File: decomposition/metav_ros_control/metav_description/urdf/sentry/sentry.gimbal.xacro (robot description, xacro)
@@ -78,5 +78,5 @@
         </joint>
     </xacro:macro>
-    <xacro:macro name="gimbal_transmission" params="prefix mechanical_reduction">
+    <xacro:macro name="gimbal_transmission" params="prefix mechanical_reduction can_network motor_id">
         <!-- <transmission name="${prefix}_gimbal_trans">
             <plugin>transmission_interface/SimpleTransmission</plugin>
@@ -97,5 +97,5 @@
             <param name="can_network_name">${can_network}</param>
             <param name="motor_id">${motor_id}</param>
-            <param name="mechanical_reduction" value="${mechanical_reduction}"/>
+            <param name="mechanical_reduction">${mechanical_reduction}</param>
         </joint>
     </xacro:macro>

File: decomposition/metav_ros_control/metav_description/urdf/sentry/sentry.xacro (robot description, xacro)
@@ -13,6 +13,6 @@
     <xacro:include filename="$(find metav_description)/urdf/sentry/sentry.chassis.xacro" />
     <xacro:chassis roller_type="$(arg roller_type)" />
-    <!-- <xacro:include filename="$(find metav_description)/urdf/sentry/sentry.gimbal.xacro" /> -->
-    <!-- <xacro:gimbal /> -->
+    <xacro:include filename="$(find metav_description)/urdf/sentry/sentry.gimbal.xacro" />
+    <xacro:gimbal />
     <!-- <xacro:include filename="$(find metav_description)/urdf/common/sensor_imu.xacro" /> -->
     <!-- <xacro:sensor_imu connected_to="pitch_gimbal" imu_name="gimbal_imu" xyz="0 0 0.1" /> -->
@@ -36,6 +36,8 @@
         <xacro:wheel_transmission prefix="back" mechanical_reduction="20.0" can_network="can1"
             motor_id="2" />
-        <!-- <xacro:gimbal_transmission prefix="yaw" mechanical_reduction="1.0"/>
-        <xacro:gimbal_transmission prefix="pitch" mechanical_reduction="1.0"/> -->
+        <xacro:gimbal_transmission prefix="yaw" mechanical_reduction="1.0" can_network="can1"
+            motor_id="5"/>
+        <xacro:gimbal_transmission prefix="pitch" mechanical_reduction="1.0" can_network="can1"
+            motor_id="6"/>
     </ros2_control>
     <xacro:if value="$(arg is_simulation)">
