Commit message: Fix launch issue

File: decomposition/metav_ros_control/metav_description/urdf/playground/single_motor.xacro (robot description, xacro)
@@ -1,93 +1,93 @@
 <?xml version="1.0"?>
 <robot name="single_motor" xmlns:xacro="http://www.ros.org/wiki/xacro">
-    <xacro:arg name="is_simulation" default="true"/>
-    <xacro:arg name="roller_type" default="simple"/>
+    <xacro:arg name="is_simulation" default="true" />
+    <xacro:arg name="roller_type" default="simple" />
     <link name="base_footprint">
     </link>
     <!-- raise the robot a bit higher to prevent it from stucking in the ground -->
     <joint name="joint_base_to_footprint" type="fixed">
-        <origin rpy="0 0 0.2" xyz="0 0 0"/>
-        <parent link="base_footprint"/>
-        <child link="base_link"/>
+        <origin rpy="0 0 0.2" xyz="0 0 0" />
+        <parent link="base_footprint" />
+        <child link="base_link" />
     </joint>
     <link name="base_link">
         <inertial>
-            <mass value="12.326"/>
-            <origin xyz="-0.000932  -0.000668  -0.01"/>
+            <mass value="12.326" />
+            <origin xyz="-0.000932  -0.000668  -0.01" />
             <inertia ixx="1.924e-1" ixy="-6.458e-4" ixz="5.951352e-3" iyy="2.473e-1"
-                     iyz="-7.22e-4" izz="3.187e-1"/>
+                iyz="-7.22e-4" izz="3.187e-1" />
         </inertial>
         <visual>
-            <origin xyz="0 0 0.05" rpy="0 0 0"/>
+            <origin xyz="0 0 0.05" rpy="0 0 0" />
             <geometry>
-                <cylinder radius="0.25" length="0.1"/>
+                <cylinder radius="0.25" length="0.1" />
             </geometry>
             <material name="silver">
-                <color rgba="0.700 0.700 0.700 1.000"/>
+                <color rgba="0.700 0.700 0.700 1.000" />
             </material>
         </visual>
         <collision>
-            <origin xyz="0 0 0.05" rpy="0 0 0"/>
+            <origin xyz="0 0 0.05" rpy="0 0 0" />
             <geometry>
-                <cylinder radius="0.25" length="0.1"/>
+                <cylinder radius="0.25" length="0.1" />
             </geometry>
         </collision>
     </link>
     <joint name="motor_joint" type="continuous">
-        <origin xyz="0 0 0.1" rpy="0 0 0"/>
-        <parent link="base_link"/>
-        <child link="motor_top"/>
-        <dynamics damping="0.0" friction="0.1"/>
-        <limit effort="30" velocity="2.0"/>
-        <axis xyz="0 0 1"/>
+        <origin xyz="0 0 0.1" rpy="0 0 0" />
+        <parent link="base_link" />
+        <child link="motor_top" />
+        <dynamics damping="0.0" friction="0.1" />
+        <limit effort="30" velocity="2.0" />
+        <axis xyz="0 0 1" />
     </joint>
     <link name="motor_top">
         <inertial>
-            <mass value="12.326"/>
-            <origin xyz="-0.000932  -0.000668  -0.01"/>
+            <mass value="12.326" />
+            <origin xyz="-0.000932  -0.000668  -0.01" />
             <inertia ixx="1.924e-1" ixy="-6.458e-4" ixz="5.951352e-3" iyy="2.473e-1"
-                     iyz="-7.22e-4" izz="3.187e-1"/>
+                iyz="-7.22e-4" izz="3.187e-1" />
         </inertial>
         <visual>
-            <origin xyz="0 0 0.1" rpy="0 0 0"/>
+            <origin xyz="0 0 0.1" rpy="0 0 0" />
             <geometry>
-                <cylinder radius="0.25" length="0.2"/>
+                <cylinder radius="0.25" length="0.2" />
             </geometry>
             <material name="black">
-                <color rgba="0.000 0.000 0.000 1.000"/>
+                <color rgba="0.000 0.000 0.000 1.000" />
             </material>
         </visual>
         <collision>
-            <origin xyz="0 0 0.1" rpy="0 0 0"/>
+            <origin xyz="0 0 0.1" rpy="0 0 0" />
             <geometry>
-                <cylinder radius="0.25" length="0.2"/>
+                <cylinder radius="0.25" length="0.2" />
             </geometry>
         </collision>
     </link>
     <joint name="motor_top_indicator_joint" type="fixed">
-        <origin xyz="0.2 0 0.2" rpy="0 0 0"/>
-        <parent link="motor_top"/>
-        <child link="motor_top_indicator"/>
+        <origin xyz="0.2 0 0.2" rpy="0 0 0" />
+        <parent link="motor_top" />
+        <child link="motor_top_indicator" />
     </joint>
     <link name="motor_top_indicator">
         <inertial>
-            <mass value="12.326"/>
-            <origin xyz="-0.000932  -0.000668  -0.01"/>
+            <mass value="12.326" />
+            <origin xyz="-0.000932  -0.000668  -0.01" />
             <inertia ixx="1.924e-1" ixy="-6.458e-4" ixz="5.951352e-3" iyy="2.473e-1"
-                     iyz="-7.22e-4" izz="3.187e-1"/>
+                iyz="-7.22e-4" izz="3.187e-1" />
         </inertial>
         <visual>
-            <origin xyz="0 0 0.01" rpy="0 0 0"/>
+            <origin xyz="0 0 0.01" rpy="0 0 0" />
             <geometry>
-                <cylinder radius="0.05" length="0.02"/>
+                <cylinder radius="0.05" length="0.02" />
             </geometry>
             <material name="white">
-                <color rgba="1.000 1.000 1.000 1.000"/>
+                <color rgba="1.000 1.000 1.000 1.000" />
             </material>
         </visual>
         <collision>
-            <origin xyz="0 0 0.01" rpy="0 0 0"/>
+            <origin xyz="0 0 0.01" rpy="0 0 0" />
             <geometry>
-                <cylinder radius="0.05" length="0.02"/>
+                <cylinder radius="0.05" length="0.02" />
             </geometry>
         </collision>
@@ -105,8 +105,12 @@
         </xacro:unless>
         <joint name="motor_joint">
-            <command_interface name="effort"/>
-            <state_interface name="position"/>
-            <state_interface name="velocity"/>
-            <state_interface name="effort"/>
+            <command_interface name="effort" />
+            <state_interface name="position" />
+            <state_interface name="velocity" />
+            <state_interface name="effort" />
+            <param name="motor_vendor">DJI</param>
+            <param name="motor_model">GM6020</param>
+            <param name="can_network_name">can0</param>
+            <param name="motor_id">1</param>
         </joint>
     </ros2_control>

Commit message: Revise inertia in single_motor.xacro to make it more sensible

File: decomposition/metav_ros_control/metav_description/urdf/playground/single_motor.xacro (robot description, xacro)
@@ -11,10 +11,14 @@
         <child link="base_link" />
     </joint>
+    <xacro:macro name="cylinder_inertia" params="m r h">
+        <inertia ixx="${m*(3*r*r+h*h)/12}" ixy="0" ixz="0"
+            iyy="${m*(3*r*r+h*h)/12}" iyz="0"
+            izz="${m*r*r/2}" />
+    </xacro:macro>
     <link name="base_link">
         <inertial>
-            <mass value="12.326" />
-            <origin xyz="-0.000932  -0.000668  -0.01" />
-            <inertia ixx="1.924e-1" ixy="-6.458e-4" ixz="5.951352e-3" iyy="2.473e-1"
-                iyz="-7.22e-4" izz="3.187e-1" />
+            <mass value="10.0" />
+            <origin xyz="0 0 0.1" />
+            <xacro:cylinder_inertia m="1.0" r="0.25" h="0.1" />
         </inertial>
         <visual>
@@ -44,8 +48,7 @@
     <link name="motor_top">
         <inertial>
-            <mass value="12.326" />
-            <origin xyz="-0.000932  -0.000668  -0.01" />
-            <inertia ixx="1.924e-1" ixy="-6.458e-4" ixz="5.951352e-3" iyy="2.473e-1"
-                iyz="-7.22e-4" izz="3.187e-1" />
+            <mass value="20.0" />
+            <origin xyz="0 0 0.1" />
+            <xacro:cylinder_inertia m="20.0" r="0.25" h="0.2" />
         </inertial>
         <visual>
@@ -72,8 +75,7 @@
     <link name="motor_top_indicator">
         <inertial>
-            <mass value="12.326" />
-            <origin xyz="-0.000932  -0.000668  -0.01" />
-            <inertia ixx="1.924e-1" ixy="-6.458e-4" ixz="5.951352e-3" iyy="2.473e-1"
-                iyz="-7.22e-4" izz="3.187e-1" />
+            <mass value="1.0" />
+            <origin xyz="0 0 0.01" />
+            <xacro:cylinder_inertia m="1.0" r="0.05" h="0.02" />
         </inertial>
         <visual>

Commit message: Add a multiple motor playground and move all Gazebo related launch stuff into meta_gazebo

File: decomposition/metav_ros_control/metav_description/urdf/playground/single_motor.xacro (robot description, xacro)
@@ -2,5 +2,4 @@
 <robot name="single_motor" xmlns:xacro="http://www.ros.org/wiki/xacro">
     <xacro:arg name="is_simulation" default="true" />
-    <xacro:arg name="roller_type" default="simple" />
     <link name="base_footprint">
     </link>
@@ -11,89 +10,9 @@
         <child link="base_link" />
     </joint>
-    <xacro:macro name="cylinder_inertia" params="m r h">
-        <inertia ixx="${m*(3*r*r+h*h)/12}" ixy="0" ixz="0"
-            iyy="${m*(3*r*r+h*h)/12}" iyz="0"
-            izz="${m*r*r/2}" />
-    </xacro:macro>
-    <link name="base_link">
-        <inertial>
-            <mass value="10.0" />
-            <origin xyz="0 0 0.1" />
-            <xacro:cylinder_inertia m="1.0" r="0.25" h="0.1" />
-        </inertial>
-        <visual>
-            <origin xyz="0 0 0.05" rpy="0 0 0" />
-            <geometry>
-                <cylinder radius="0.25" length="0.1" />
-            </geometry>
-            <material name="silver">
-                <color rgba="0.700 0.700 0.700 1.000" />
-            </material>
-        </visual>
-        <collision>
-            <origin xyz="0 0 0.05" rpy="0 0 0" />
-            <geometry>
-                <cylinder radius="0.25" length="0.1" />
-            </geometry>
-        </collision>
-    </link>
-    <joint name="motor_joint" type="continuous">
-        <origin xyz="0 0 0.1" rpy="0 0 0" />
-        <parent link="base_link" />
-        <child link="motor_top" />
-        <dynamics damping="0.0" friction="0.1" />
-        <limit effort="30" velocity="2.0" />
-        <axis xyz="0 0 1" />
-    </joint>
-    <link name="motor_top">
-        <inertial>
-            <mass value="20.0" />
-            <origin xyz="0 0 0.1" />
-            <xacro:cylinder_inertia m="20.0" r="0.25" h="0.2" />
-        </inertial>
-        <visual>
-            <origin xyz="0 0 0.1" rpy="0 0 0" />
-            <geometry>
-                <cylinder radius="0.25" length="0.2" />
-            </geometry>
-            <material name="black">
-                <color rgba="0.000 0.000 0.000 1.000" />
-            </material>
-        </visual>
-        <collision>
-            <origin xyz="0 0 0.1" rpy="0 0 0" />
-            <geometry>
-                <cylinder radius="0.25" length="0.2" />
-            </geometry>
-        </collision>
-    </link>
-    <joint name="motor_top_indicator_joint" type="fixed">
-        <origin xyz="0.2 0 0.2" rpy="0 0 0" />
-        <parent link="motor_top" />
-        <child link="motor_top_indicator" />
-    </joint>
-    <link name="motor_top_indicator">
-        <inertial>
-            <mass value="1.0" />
-            <origin xyz="0 0 0.01" />
-            <xacro:cylinder_inertia m="1.0" r="0.05" h="0.02" />
-        </inertial>
-        <visual>
-            <origin xyz="0 0 0.01" rpy="0 0 0" />
-            <geometry>
-                <cylinder radius="0.05" length="0.02" />
-            </geometry>
-            <material name="white">
-                <color rgba="1.000 1.000 1.000 1.000" />
-            </material>
-        </visual>
-        <collision>
-            <origin xyz="0 0 0.01" rpy="0 0 0" />
-            <geometry>
-                <cylinder radius="0.05" length="0.02" />
-            </geometry>
-        </collision>
-    </link>
-    <ros2_control name="single_motor_control" type="system">
+    <link name="base_link" />
+    <xacro:include filename="$(find metav_description)/urdf/playground/motor.xacro" />
+    <xacro:motor name="motor" connected_to="base_link" x="0" y="0" />
+    <ros2_control
+        name="single_motor_control" type="system">
         <xacro:if value="$(arg is_simulation)">
             <hardware>
@@ -116,5 +35,6 @@
         </joint>
     </ros2_control>
-    <xacro:if value="$(arg is_simulation)">
+    <xacro:if
+        value="$(arg is_simulation)">
         <gazebo>
             <plugin filename="ign_ros2_control-system"
