Commit message: Ready for chassis control test on real hardware

File: decomposition/metav_ros_control/metav_description/urdf/common/omni_wheel.xacro (robot description, xacro)
@@ -1,12 +1,12 @@
 <?xml version="1.0"?>
 <robot name="omni_wheel" xmlns:xacro="http://www.ros.org/wiki/xacro">
-    <xacro:property name="wheel_radius" value="0.0762"/>
-    <xacro:property name="roller_radius" value="0.009"/>
+    <xacro:property name="wheel_radius" value="0.0762" />
+    <xacro:property name="roller_radius" value="0.009" />
     <xacro:macro name="roller" params="prefix suffix theta roller_type">
         <xacro:if value="${suffix % 2 == 1}">
-            <xacro:property name="joint_y_offset" value="0.009563"/>
+            <xacro:property name="joint_y_offset" value="0.009563" />
         </xacro:if>
         <xacro:if value="${suffix % 2 == 0}">
-            <xacro:property name="joint_y_offset" value="-0.009563"/>
+            <xacro:property name="joint_y_offset" value="-0.009563" />
         </xacro:if>
         <!--  link  -->
@@ -14,48 +14,50 @@
             <xacro:if value="${roller_type=='simple'}">
                 <visual>
-                    <origin xyz="0 0 0" rpy="0 0 0"/>
+                    <origin xyz="0 0 0" rpy="0 0 0" />
                     <geometry>
-                        <mesh filename="file://$(find metav_description)/meshes/common/omni_roller.stl"
-                              scale="0.001 0.001 0.001"/>
+                        <mesh
+                            filename="file://$(find metav_description)/meshes/common/omni_roller.stl"
+                            scale="0.001 0.001 0.001" />
                     </geometry>
                     <material name="black">
-                        <color rgba="0.000 0.000 0.000 1.000"/>
+                        <color rgba="0.000 0.000 0.000 1.000" />
                     </material>
                 </visual>
                 <collision>
                     <geometry>
-                        <sphere radius="${roller_radius}"/>
+                        <sphere radius="${roller_radius}" />
                     </geometry>
                 </collision>
                 <collision>
-                    <origin rpy="0 1.57 0" xyz="0 0 0"/>
+                    <origin rpy="0 1.57 0" xyz="0 0 0" />
                     <geometry>
-                        <cylinder length="19e-3" radius="8.6e-3"/>
+                        <cylinder length="19e-3" radius="8.6e-3" />
                     </geometry>
                 </collision>
             </xacro:if>
             <inertial>
-                <mass value="0.0058"/>
-                <inertia ixx="270.867e-9" ixy="1.547e-19" ixz="2.133e-19" iyy="291.412e-9" iyz="0.0" izz="291.412e-9"/>
+                <mass value="0.0058" />
+                <inertia ixx="270.867e-9" ixy="1.547e-19" ixz="2.133e-19" iyy="291.412e-9" iyz="0.0"
+                    izz="291.412e-9" />
             </inertial>
         </link>
         <joint name="${prefix}_roller_${suffix}_joint" type="continuous">
             <origin
-                    xyz="${(wheel_radius-roller_radius)*cos(theta-pi/2)} ${joint_y_offset} ${(wheel_radius-roller_radius)*sin(theta-pi/2)}"
-                    rpy="0 ${-theta} 0"/>
-            <axis xyz="1 0 0"/>
-            <dynamics damping="0.0" friction="0.001"/>
-            <parent link="${prefix}_wheel"/>
-            <child link="${prefix}_roller_${suffix}"/>
+                xyz="${(wheel_radius-roller_radius)*cos(theta-pi/2)} ${joint_y_offset} ${(wheel_radius-roller_radius)*sin(theta-pi/2)}"
+                rpy="0 ${-theta} 0" />
+            <axis xyz="1 0 0" />
+            <dynamics damping="0.0" friction="0.001" />
+            <parent link="${prefix}_wheel" />
+            <child link="${prefix}_roller_${suffix}" />
         </joint>
         <gazebo reference="${prefix}_roller_${suffix}">
-            <mu1 value="2000.0"/>
-            <mu2 value="2000.0"/>
-            <kp value="1000000.0"/>
-            <kd value="100.0"/>
+            <mu1 value="2000.0" />
+            <mu2 value="2000.0" />
+            <kp value="1000000.0" />
+            <kd value="100.0" />
         </gazebo>
     </xacro:macro>
     <xacro:macro name="omni_wheel"
-                 params="prefix connected_to wheel_x_offset wheel_y_offset wheel_z_offset rotation_degree roller_type max_effort max_velocity">
+        params="prefix connected_to wheel_x_offset wheel_y_offset wheel_z_offset rotation_degree roller_type max_effort max_velocity">
         <!--  link  -->
         <link name="${prefix}_wheel">
@@ -63,58 +65,85 @@
                 <geometry>
                     <mesh filename="file://$(find metav_description)/meshes/common/omni_wheel.stl"
-                          scale="0.001 0.001 0.001"/>
+                        scale="0.001 0.001 0.001" />
                 </geometry>
                 <material name="gray">
-                    <color rgba="0.250 0.250 0.250 1.000"/>
+                    <color rgba="0.250 0.250 0.250 1.000" />
                 </material>
             </visual>
             <inertial>
-                <mass value="0.59"/>
-                <inertia ixx="1.416e-3" ixy="0.0" ixz="0.0" iyy="2.749e-3" iyz="0.0" izz="1.416e-3"/>
+                <mass value="0.59" />
+                <inertia ixx="1.416e-3" ixy="0.0" ixz="0.0" iyy="2.749e-3" iyz="0.0" izz="1.416e-3" />
             </inertial>
         </link>
         <!--  joint  -->
         <joint name="${prefix}_wheel_joint" type="continuous">
-            <axis xyz="0 1 0"/>
-            <origin xyz="${wheel_x_offset} ${wheel_y_offset} ${wheel_offset_z}" rpy="0 0 ${rotation_degree}"/>
+            <axis xyz="0 1 0" />
+            <origin xyz="${wheel_x_offset} ${wheel_y_offset} ${wheel_offset_z}"
+                rpy="0 0 ${rotation_degree}" />
             <!--      limit not work while type="continuous"-->
-            <limit effort="${max_effort}" velocity="${max_velocity}" lower="-1e9" upper="1e9"/>
-            <dynamics damping="0.0" friction="0.05"/>
-            <parent link="${connected_to}"/>
-            <child link="${prefix}_wheel"/>
+            <limit effort="${max_effort}" velocity="${max_velocity}" lower="-1e9" upper="1e9" />
+            <dynamics damping="0.0" friction="0.05" />
+            <parent link="${connected_to}" />
+            <child link="${prefix}_wheel" />
         </joint>
         <xacro:unless value="${roller_type=='none'}">
-            <xacro:roller prefix="${prefix}" suffix="0" theta="${0*pi/13}" roller_type="${roller_type}"/>
-            <xacro:roller prefix="${prefix}" suffix="1" theta="${1*pi/13}" roller_type="${roller_type}"/>
-            <xacro:roller prefix="${prefix}" suffix="2" theta="${2*pi/13}" roller_type="${roller_type}"/>
-            <xacro:roller prefix="${prefix}" suffix="3" theta="${3*pi/13}" roller_type="${roller_type}"/>
-            <xacro:roller prefix="${prefix}" suffix="4" theta="${4*pi/13}" roller_type="${roller_type}"/>
-            <xacro:roller prefix="${prefix}" suffix="5" theta="${5*pi/13}" roller_type="${roller_type}"/>
-            <xacro:roller prefix="${prefix}" suffix="6" theta="${6*pi/13}" roller_type="${roller_type}"/>
-            <xacro:roller prefix="${prefix}" suffix="7" theta="${7*pi/13}" roller_type="${roller_type}"/>
-            <xacro:roller prefix="${prefix}" suffix="8" theta="${8*pi/13}" roller_type="${roller_type}"/>
-            <xacro:roller prefix="${prefix}" suffix="9" theta="${9*pi/13}" roller_type="${roller_type}"/>
-            <xacro:roller prefix="${prefix}" suffix="10" theta="${10*pi/13}" roller_type="${roller_type}"/>
-            <xacro:roller prefix="${prefix}" suffix="11" theta="${11*pi/13}" roller_type="${roller_type}"/>
-            <xacro:roller prefix="${prefix}" suffix="12" theta="${12*pi/13}" roller_type="${roller_type}"/>
-            <xacro:roller prefix="${prefix}" suffix="13" theta="${13*pi/13}" roller_type="${roller_type}"/>
-            <xacro:roller prefix="${prefix}" suffix="14" theta="${14*pi/13}" roller_type="${roller_type}"/>
-            <xacro:roller prefix="${prefix}" suffix="15" theta="${15*pi/13}" roller_type="${roller_type}"/>
-            <xacro:roller prefix="${prefix}" suffix="16" theta="${16*pi/13}" roller_type="${roller_type}"/>
-            <xacro:roller prefix="${prefix}" suffix="17" theta="${17*pi/13}" roller_type="${roller_type}"/>
-            <xacro:roller prefix="${prefix}" suffix="18" theta="${18*pi/13}" roller_type="${roller_type}"/>
-            <xacro:roller prefix="${prefix}" suffix="19" theta="${19*pi/13}" roller_type="${roller_type}"/>
-            <xacro:roller prefix="${prefix}" suffix="20" theta="${20*pi/13}" roller_type="${roller_type}"/>
-            <xacro:roller prefix="${prefix}" suffix="21" theta="${21*pi/13}" roller_type="${roller_type}"/>
-            <xacro:roller prefix="${prefix}" suffix="22" theta="${22*pi/13}" roller_type="${roller_type}"/>
-            <xacro:roller prefix="${prefix}" suffix="23" theta="${23*pi/13}" roller_type="${roller_type}"/>
-            <xacro:roller prefix="${prefix}" suffix="24" theta="${24*pi/13}" roller_type="${roller_type}"/>
-            <xacro:roller prefix="${prefix}" suffix="25" theta="${25*pi/13}" roller_type="${roller_type}"/>
+            <xacro:roller prefix="${prefix}" suffix="0" theta="${0*pi/13}"
+                roller_type="${roller_type}" />
+            <xacro:roller prefix="${prefix}" suffix="1" theta="${1*pi/13}"
+                roller_type="${roller_type}" />
+            <xacro:roller prefix="${prefix}" suffix="2" theta="${2*pi/13}"
+                roller_type="${roller_type}" />
+            <xacro:roller prefix="${prefix}" suffix="3" theta="${3*pi/13}"
+                roller_type="${roller_type}" />
+            <xacro:roller prefix="${prefix}" suffix="4" theta="${4*pi/13}"
+                roller_type="${roller_type}" />
+            <xacro:roller prefix="${prefix}" suffix="5" theta="${5*pi/13}"
+                roller_type="${roller_type}" />
+            <xacro:roller prefix="${prefix}" suffix="6" theta="${6*pi/13}"
+                roller_type="${roller_type}" />
+            <xacro:roller prefix="${prefix}" suffix="7" theta="${7*pi/13}"
+                roller_type="${roller_type}" />
+            <xacro:roller prefix="${prefix}" suffix="8" theta="${8*pi/13}"
+                roller_type="${roller_type}" />
+            <xacro:roller prefix="${prefix}" suffix="9" theta="${9*pi/13}"
+                roller_type="${roller_type}" />
+            <xacro:roller prefix="${prefix}" suffix="10" theta="${10*pi/13}"
+                roller_type="${roller_type}" />
+            <xacro:roller prefix="${prefix}" suffix="11" theta="${11*pi/13}"
+                roller_type="${roller_type}" />
+            <xacro:roller prefix="${prefix}" suffix="12" theta="${12*pi/13}"
+                roller_type="${roller_type}" />
+            <xacro:roller prefix="${prefix}" suffix="13" theta="${13*pi/13}"
+                roller_type="${roller_type}" />
+            <xacro:roller prefix="${prefix}" suffix="14" theta="${14*pi/13}"
+                roller_type="${roller_type}" />
+            <xacro:roller prefix="${prefix}" suffix="15" theta="${15*pi/13}"
+                roller_type="${roller_type}" />
+            <xacro:roller prefix="${prefix}" suffix="16" theta="${16*pi/13}"
+                roller_type="${roller_type}" />
+            <xacro:roller prefix="${prefix}" suffix="17" theta="${17*pi/13}"
+                roller_type="${roller_type}" />
+            <xacro:roller prefix="${prefix}" suffix="18" theta="${18*pi/13}"
+                roller_type="${roller_type}" />
+            <xacro:roller prefix="${prefix}" suffix="19" theta="${19*pi/13}"
+                roller_type="${roller_type}" />
+            <xacro:roller prefix="${prefix}" suffix="20" theta="${20*pi/13}"
+                roller_type="${roller_type}" />
+            <xacro:roller prefix="${prefix}" suffix="21" theta="${21*pi/13}"
+                roller_type="${roller_type}" />
+            <xacro:roller prefix="${prefix}" suffix="22" theta="${22*pi/13}"
+                roller_type="${roller_type}" />
+            <xacro:roller prefix="${prefix}" suffix="23" theta="${23*pi/13}"
+                roller_type="${roller_type}" />
+            <xacro:roller prefix="${prefix}" suffix="24" theta="${24*pi/13}"
+                roller_type="${roller_type}" />
+            <xacro:roller prefix="${prefix}" suffix="25" theta="${25*pi/13}"
+                roller_type="${roller_type}" />
         </xacro:unless>
     </xacro:macro>
-    <xacro:macro name="wheel_transmission" params="prefix mechanical_reduction">
+    <xacro:macro name="wheel_transmission" params="prefix mechanical_reduction can_network motor_id">
         <transmission name="${prefix}_wheel_trans">
             <plugin>transmission_interface/SimpleTransmission</plugin>
-            <actuator name="${prefix}_wheel_motor" role="${prefix}_wheel_motor"/>
+            <actuator name="${prefix}_wheel_motor" role="${prefix}_wheel_motor" />
             <joint name="${prefix}_wheel_joint" role="${prefix}_wheel_joint">
                 <mechanical_reduction>${mechanical_reduction}</mechanical_reduction>
@@ -125,7 +154,11 @@
             <command_interface name="effort">
             </command_interface>
-            <state_interface name="position"/>
-            <state_interface name="velocity"/>
-            <state_interface name="effort"/>
+            <state_interface name="position" />
+            <state_interface name="velocity" />
+            <state_interface name="effort" />
+            <param name="motor_vendor">DJI</param>
+            <param name="motor_model">M3508</param>
+            <param name="can_network_name">${can_network}</param>
+            <param name="motor_id">${motor_id}</param>
         </joint>
     </xacro:macro>

File: decomposition/metav_ros_control/metav_description/urdf/sentry/sentry.xacro (robot description, xacro)
@@ -1,20 +1,20 @@
 <?xml version="1.0"?>
 <robot name="sentry" xmlns:xacro="http://www.ros.org/wiki/xacro">
-    <xacro:arg name="is_simulation" default="true"/>
-    <xacro:arg name="roller_type" default="simple"/>
+    <xacro:arg name="is_simulation" default="true" />
+    <xacro:arg name="roller_type" default="simple" />
     <link name="base_footprint">
     </link>
     <!-- raise the robot a bit higher to prevent it from stucking in the ground -->
     <joint name="joint_base_to_footprint" type="fixed">
-        <origin rpy="0 0 0" xyz="0 0 1"/>
-        <parent link="base_footprint"/>
-        <child link="base_link"/>
+        <origin rpy="0 0 0" xyz="0 0 1" />
+        <parent link="base_footprint" />
+        <child link="base_link" />
     </joint>
-    <xacro:include filename="$(find metav_description)/urdf/sentry/sentry.chassis.xacro"/>
-    <xacro:chassis roller_type="$(arg roller_type)"/>
-    <xacro:include filename="$(find metav_description)/urdf/sentry/sentry.gimbal.xacro"/>
-    <xacro:gimbal/>
-    <xacro:include filename="$(find metav_description)/urdf/common/sensor_imu.xacro"/>
-    <xacro:sensor_imu connected_to="pitch_gimbal" imu_name="gimbal_imu" xyz="0 0 0.1"/>
+    <xacro:include filename="$(find metav_description)/urdf/sentry/sentry.chassis.xacro" />
+    <xacro:chassis roller_type="$(arg roller_type)" />
+    <!-- <xacro:include filename="$(find metav_description)/urdf/sentry/sentry.gimbal.xacro" /> -->
+    <!-- <xacro:gimbal /> -->
+    <!-- <xacro:include filename="$(find metav_description)/urdf/common/sensor_imu.xacro" /> -->
+    <!-- <xacro:sensor_imu connected_to="pitch_gimbal" imu_name="gimbal_imu" xyz="0 0 0.1" /> -->
     <ros2_control name="sentry_control" type="system">
         <xacro:if value="$(arg is_simulation)">
@@ -23,13 +23,22 @@
             </hardware>
         </xacro:if>
-        <xacro:wheel_transmission prefix="front" mechanical_reduction="20.0"/>
-        <xacro:wheel_transmission prefix="right" mechanical_reduction="20.0"/>
-        <xacro:wheel_transmission prefix="left" mechanical_reduction="20.0"/>
-        <xacro:wheel_transmission prefix="back" mechanical_reduction="20.0"/>
-        <xacro:gimbal_transmission prefix="yaw" mechanical_reduction="1.0"/>
-        <xacro:gimbal_transmission prefix="pitch" mechanical_reduction="1.0"/>
+        <xacro:unless value="$(arg is_simulation)">
+            <hardware>
+                <plugin>metav_hardware/MetavRobotHardwareInterface</plugin>
+            </hardware>
+        </xacro:unless>
+        <xacro:wheel_transmission prefix="front" mechanical_reduction="20.0" can_network="can0"
+            motor_id="1" />
+        <xacro:wheel_transmission prefix="right" mechanical_reduction="20.0" can_network="can0"
+            motor_id="3" />
+        <xacro:wheel_transmission prefix="left" mechanical_reduction="20.0" can_network="can0"
+            motor_id="4" />
+        <xacro:wheel_transmission prefix="back" mechanical_reduction="20.0" can_network="can0"
+            motor_id="2" />
+        <!-- <xacro:gimbal_transmission prefix="yaw" mechanical_reduction="1.0"/>
+        <xacro:gimbal_transmission prefix="pitch" mechanical_reduction="1.0"/> -->
     </ros2_control>
     <xacro:if value="$(arg is_simulation)">
-        <xacro:include filename="$(find metav_description)/urdf/sentry/sentry.gazebo.xacro"/>
+        <xacro:include filename="$(find metav_description)/urdf/sentry/sentry.gazebo.xacro" />
     </xacro:if>
 </robot>
