Commit message: Revise urdf to conform hardware interface changes

File: decomposition/metav_ros_control/metav_description/urdf/common/omni_wheel.xacro (robot description, xacro)
@@ -159,5 +159,4 @@
             <param name="motor_vendor">DJI</param>
             <param name="motor_model">M3508</param>
-            <param name="can_network_name">${can_network}</param>
             <param name="motor_id">${motor_id}</param>
             <param name="mechanical_reduction">${mechanical_reduction}</param>

File: decomposition/metav_ros_control/metav_description/urdf/playground/single_motor.xacro (robot description, xacro)
@@ -101,5 +101,7 @@
         <xacro:unless value="$(arg is_simulation)">
             <hardware>
-                <plugin>metav_hardware/MetavRobotHardwareInterface</plugin>
+                <plugin>meta_hardware/MetaRobotMotorNetwork</plugin>
+                <param name="vendor" value="DJI" />
+                <param name="can_network_name" value="can0" />
             </hardware>
         </xacro:unless>
@@ -111,5 +113,4 @@
             <param name="motor_vendor">DJI</param>
             <param name="motor_model">GM6020</param>
-            <param name="can_network_name">can0</param>
             <param name="motor_id">1</param>
         </joint>

File: decomposition/metav_ros_control/metav_description/urdf/sentry/sentry.gimbal.xacro (robot description, xacro)
@@ -1,28 +1,30 @@
 <?xml version="1.0"?>
 <robot name="sentry" xmlns:xacro="http://www.ros.org/wiki/xacro">
-    <xacro:property name="threshold" value="0.08"/>
-    <xacro:property name="pitch_lower_limit" value="-0.72"/>
-    <xacro:property name="pitch_upper_limit" value="0.457"/>
+    <xacro:property name="threshold" value="0.08" />
+    <xacro:property name="pitch_lower_limit" value="-0.72" />
+    <xacro:property name="pitch_upper_limit" value="0.457" />
     <xacro:macro name="gimbal" params="">
         <link name="yaw_gimbal">
             <inertial>
-                <mass value="0.2"/>
-                <origin xyz="0 0 0"/>
+                <mass value="0.2" />
+                <origin xyz="0 0 0" />
                 <inertia ixx="4.878e-4" ixy="1.941e-5" ixz="2.44e-4" iyy="8.322e-4"
-                        iyz="-1.812e-5" izz="4.513e-4"/>
+                    iyz="-1.812e-5" izz="4.513e-4" />
             </inertial>
             <visual>
-                <origin xyz="0 0 0" rpy="0 0 0"/>
+                <origin xyz="0 0 0" rpy="0 0 0" />
                 <geometry>
-                    <mesh filename="file://$(find metav_description)/meshes/sentry/yaw_gimbal.stl" scale="0.001 0.001 0.001"/>
+                    <mesh filename="file://$(find metav_description)/meshes/sentry/yaw_gimbal.stl"
+                        scale="0.001 0.001 0.001" />
                 </geometry>
                 <material name="silver">
-                    <color rgba="0.700 0.700 0.700 1.000"/>
+                    <color rgba="0.700 0.700 0.700 1.000" />
                 </material>
             </visual>
             <collision>
-                <origin xyz="0 0 0" rpy="0 0 0"/>
+                <origin xyz="0 0 0" rpy="0 0 0" />
                 <geometry>
-                    <mesh filename="file://$(find metav_description)/meshes/sentry/yaw_gimbal.stl" scale="0.001 0.001 0.001"/>
+                    <mesh filename="file://$(find metav_description)/meshes/sentry/yaw_gimbal.stl"
+                        scale="0.001 0.001 0.001" />
                 </geometry>
             </collision>
@@ -30,53 +32,57 @@
         <joint name="yaw_gimbal_joint" type="continuous">
             <origin xyz="0 0 0.162"
-                    rpy="0 0 0"/>
-            <dynamics damping="0.0" friction="0.1"/>
-            <limit effort="1.2" velocity="31"/>
-            <parent link="base_link"/>
-            <child link="yaw_gimbal"/>
-            <axis xyz="0 0 1"/>
+                rpy="0 0 0" />
+            <dynamics damping="0.0" friction="0.1" />
+            <limit effort="1.2" velocity="31" />
+            <parent link="base_link" />
+            <child link="yaw_gimbal" />
+            <axis xyz="0 0 1" />
         </joint>
-        <link name="supply_frame"/>
+        <link name="supply_frame" />
         <joint name="supply_joint" type="fixed">
-            <origin xyz="0 0 0" rpy="0 0 ${pi/3}"/>
-            <parent link="yaw_gimbal"/>
-            <child link="supply_frame"/>
+            <origin xyz="0 0 0" rpy="0 0 ${pi/3}" />
+            <parent link="yaw_gimbal" />
+            <child link="supply_frame" />
         </joint>
         <link name="pitch_gimbal">
             <inertial>
-                <mass value="0.644"/>
-                <origin xyz="0.029 0.000617 0.0376"/>
+                <mass value="0.644" />
+                <origin xyz="0.029 0.000617 0.0376" />
                 <inertia ixx="1.8216e-3" ixy="5.514e-6" ixz="1.58e-4" iyy="5.68e-3"
-                        iyz="-6.628e-6" izz="4.396e-3"/>
+                    iyz="-6.628e-6" izz="4.396e-3" />
             </inertial>
             <visual>
-                <origin xyz="0 0 0" rpy="0 0 0"/>
+                <origin xyz="0 0 0" rpy="0 0 0" />
                 <geometry>
-                    <mesh filename="file://$(find metav_description)/meshes/sentry/pitch_gimbal.stl" scale="0.001 0.001 0.001"/>
+                    <mesh filename="file://$(find metav_description)/meshes/sentry/pitch_gimbal.stl"
+                        scale="0.001 0.001 0.001" />
                 </geometry>
                 <material name="silver">
-                    <color rgba="0.700 0.700 0.700 1.000"/>
+                    <color rgba="0.700 0.700 0.700 1.000" />
                 </material>
             </visual>
             <collision>
-                <origin xyz="0 0 0" rpy="0 0 0"/>
+                <origin xyz="0 0 0" rpy="0 0 0" />
                 <geometry>
-                    <mesh filename="file://$(find metav_description)/meshes/sentry/pitch_gimbal.stl" scale="0.001 0.001 0.001"/>
+                    <mesh filename="file://$(find metav_description)/meshes/sentry/pitch_gimbal.stl"
+                        scale="0.001 0.001 0.001" />
                 </geometry>
             </collision>
         </link>
         <joint name="pitch_gimbal_joint" type="revolute">
-            <origin xyz="-0.029 0 0.257" rpy="0 0 0"/>
-            <dynamics damping="0.0" friction="0.1"/>
-            <limit effort="3." velocity="86" lower="${pitch_lower_limit}" upper="${pitch_upper_limit}"/>
+            <origin xyz="-0.029 0 0.257" rpy="0 0 0" />
+            <dynamics damping="0.0" friction="0.1" />
+            <limit effort="3." velocity="86" lower="${pitch_lower_limit}"
+                upper="${pitch_upper_limit}" />
             <safety_controller k_position="100" k_velocity="0.1"
-                            soft_lower_limit="${pitch_lower_limit+threshold}"
-                            soft_upper_limit="${pitch_upper_limit-threshold}"/>
-            <parent link="yaw_gimbal"/>
-            <child link="pitch_gimbal"/>
-            <axis xyz="0 1 0 "/>
+                soft_lower_limit="${pitch_lower_limit+threshold}"
+                soft_upper_limit="${pitch_upper_limit-threshold}" />
+            <parent link="yaw_gimbal" />
+            <child link="pitch_gimbal" />
+            <axis xyz="0 1 0 " />
         </joint>
     </xacro:macro>
-    <xacro:macro name="gimbal_transmission" params="prefix mechanical_reduction can_network motor_id">
+    <xacro:macro name="gimbal_transmission"
+        params="prefix mechanical_reduction can_network motor_id">
         <!-- <transmission name="${prefix}_gimbal_trans">
             <plugin>transmission_interface/SimpleTransmission</plugin>
@@ -88,12 +94,9 @@
         </transmission> -->
         <joint name="${prefix}_gimbal_joint">
-            <command_interface name="effort">
-            </command_interface>
-            <state_interface name="position"/>
-            <state_interface name="velocity"/>
-            <state_interface name="effort"/>
-            <param name="motor_vendor">DJI</param>
+            <command_interface name="effort" />
+            <state_interface name="position" />
+            <state_interface name="velocity" />
+            <state_interface name="effort" />
             <param name="motor_model">GM6020</param>
-            <param name="can_network_name">${can_network}</param>
             <param name="motor_id">${motor_id}</param>
             <param name="mechanical_reduction">${mechanical_reduction}</param>

File: decomposition/metav_ros_control/metav_description/urdf/sentry/sentry.xacro (robot description, xacro)
@@ -16,31 +16,49 @@
     <xacro:gimbal />
     <xacro:include filename="$(find metav_description)/urdf/common/sensor_imu.xacro" />
-    <xacro:sensor_imu connected_to="pitch_gimbal" imu_name="gimbal_imu" xyz="0 0 0.1" rpy="3.14159 0 0" />
+    <xacro:sensor_imu connected_to="pitch_gimbal" imu_name="gimbal_imu" xyz="0 0 0.1"
+        rpy="3.14159 0 0" />
     <xacro:include filename="$(find metav_description)/urdf/common/sensor_mid360.xacro" />
-    <xacro:sensor_mid360 connected_to="yaw_gimbal" name="livox_frame" xyz="0.1687 0 0.11" rpy="0 0.2269 0" />
-    <ros2_control name="sentry_control" type="system">
-        <xacro:if value="$(arg is_simulation)">
+    <xacro:sensor_mid360 connected_to="yaw_gimbal" name="livox_frame" xyz="0.1687 0 0.11"
+        rpy="0 0.2269 0" />
+    <xacro:unless value="$(arg is_simulation)">
+        <ros2_control name="dji_motors" type="system">
+            <hardware>
+                <plugin>meta_hardware/MetaRobotMotorNetwork</plugin>
+                <param name="vendor" value="DJI" />
+                <param name="can_network_name" value="can1" />
+            </hardware>
+            <xacro:wheel_transmission prefix="front" mechanical_reduction="20.0" can_network="can1"
+                motor_id="1" />
+            <xacro:wheel_transmission prefix="right" mechanical_reduction="20.0" can_network="can1"
+                motor_id="3" />
+            <xacro:wheel_transmission prefix="left" mechanical_reduction="20.0" can_network="can1"
+                motor_id="4" />
+            <xacro:wheel_transmission prefix="back" mechanical_reduction="20.0" can_network="can1"
+                motor_id="2" />
+            <xacro:gimbal_transmission prefix="yaw" mechanical_reduction="1.0" can_network="can1"
+                motor_id="5" />
+            <xacro:gimbal_transmission prefix="pitch" mechanical_reduction="-1.0" can_network="can1"
+                motor_id="6" />
+        </ros2_control>
+    </xacro:unless>
+    <xacro:if value="$(arg is_simulation)">
+        <ros2_control name="sentry_control" type="system">
             <hardware>
                 <plugin>ign_ros2_control/IgnitionSystem</plugin>
             </hardware>
-        </xacro:if>
-        <xacro:unless value="$(arg is_simulation)">
-            <hardware>
-                <plugin>metav_hardware/MetavRobotHardwareInterface</plugin>
-            </hardware>
-        </xacro:unless>
-        <xacro:wheel_transmission prefix="front" mechanical_reduction="20.0" can_network="can1"
-            motor_id="1" />
-        <xacro:wheel_transmission prefix="right" mechanical_reduction="20.0" can_network="can1"
-            motor_id="3" />
-        <xacro:wheel_transmission prefix="left" mechanical_reduction="20.0" can_network="can1"
-            motor_id="4" />
-        <xacro:wheel_transmission prefix="back" mechanical_reduction="20.0" can_network="can1"
-            motor_id="2" />
-        <xacro:gimbal_transmission prefix="yaw" mechanical_reduction="1.0" can_network="can1"
-            motor_id="5"/>
-        <xacro:gimbal_transmission prefix="pitch" mechanical_reduction="-1.0" can_network="can1"
-            motor_id="6"/>
-    </ros2_control>
+            <xacro:wheel_transmission prefix="front" mechanical_reduction="20.0" can_network="can1"
+                motor_id="1" />
+            <xacro:wheel_transmission prefix="right" mechanical_reduction="20.0" can_network="can1"
+                motor_id="3" />
+            <xacro:wheel_transmission prefix="left" mechanical_reduction="20.0" can_network="can1"
+                motor_id="4" />
+            <xacro:wheel_transmission prefix="back" mechanical_reduction="20.0" can_network="can1"
+                motor_id="2" />
+            <xacro:gimbal_transmission prefix="yaw" mechanical_reduction="1.0" can_network="can1"
+                motor_id="5" />
+            <xacro:gimbal_transmission prefix="pitch" mechanical_reduction="-1.0" can_network="can1"
+                motor_id="6" />
+        </ros2_control>
+    </xacro:if>
     <xacro:if value="$(arg is_simulation)">
         <xacro:include filename="$(find metav_description)/urdf/sentry/sentry.gazebo.xacro" />

Commit message: Put joint and motor offset calculation into hardware interface, simplifying controller side code.

File: decomposition/metav_ros_control/metav_description/urdf/common/omni_wheel.xacro (robot description, xacro)
@@ -157,8 +157,8 @@
             <state_interface name="velocity" />
             <state_interface name="effort" />
-            <param name="motor_vendor">DJI</param>
             <param name="motor_model">M3508</param>
             <param name="motor_id">${motor_id}</param>
             <param name="mechanical_reduction">${mechanical_reduction}</param>
+            <param name="offset">0.0</param>
         </joint>
     </xacro:macro>

File: decomposition/metav_ros_control/metav_description/urdf/playground/multiple_motors.xacro (robot description, xacro)
@@ -6,5 +6,5 @@
     <!-- raise the robot a bit higher to prevent it from stucking in the ground -->
     <joint name="joint_base_to_footprint" type="fixed">
-        <origin rpy="0 0 0.2" xyz="0 0 0" />
+        <origin rpy="0 0 0" xyz="0 0 0.2" />
         <parent link="base_footprint" />
         <child link="base_link" />
@@ -49,4 +49,5 @@
                 <param name="motor_id">1</param>
                 <param name="mechanical_reduction">1.0</param>
+                <param name="offset">0.0</param>
             </joint>
         </ros2_control>
@@ -65,4 +66,5 @@
                 <param name="motor_id">1</param>
                 <param name="mechanical_reduction">1.0</param>
+                <param name="offset">0.0</param>
                 <param name="Kp">30.0</param>
                 <param name="Kd">1.0</param>

File: decomposition/metav_ros_control/metav_description/urdf/playground/single_motor.xacro (robot description, xacro)
@@ -6,5 +6,5 @@
     <!-- raise the robot a bit higher to prevent it from stucking in the ground -->
     <joint name="joint_base_to_footprint" type="fixed">
-        <origin rpy="0 0 0.2" xyz="0 0 0" />
+        <origin rpy="0 0 0" xyz="0 0 0.2" />
         <parent link="base_footprint" />
         <child link="base_link" />
@@ -34,4 +34,5 @@
             <param name="motor_id">1</param>
             <param name="mechanical_reduction">1.0</param>
+            <param name="offset">0.0</param>
         </joint>
     </ros2_control>

File: decomposition/metav_ros_control/metav_description/urdf/sentry/sentry.gimbal.xacro (robot description, xacro)
@@ -84,13 +84,5 @@
     </xacro:macro>
     <xacro:macro name="gimbal_transmission"
-        params="prefix mechanical_reduction can_network motor_id">
-        <!-- <transmission name="${prefix}_gimbal_trans">
-            <plugin>transmission_interface/SimpleTransmission</plugin>
-            <actuator name="${prefix}_gimbal_motor" role="${prefix}_gimbal_motor"/>
-            <joint name="${prefix}_gimbal_joint" role="${prefix}_gimbal_joint">
-                <mechanical_reduction>${mechanical_reduction}</mechanical_reduction>
-                <offset>0.0</offset>
-            </joint>
-        </transmission> -->
+        params="prefix mechanical_reduction offset can_network motor_id">
         <joint name="${prefix}_gimbal_joint">
             <command_interface name="effort" />
@@ -101,4 +93,5 @@
             <param name="motor_id">${motor_id}</param>
             <param name="mechanical_reduction">${mechanical_reduction}</param>
+            <param name="offset">${offset}</param>
         </joint>
     </xacro:macro>

File: decomposition/metav_ros_control/metav_description/urdf/sentry/sentry.xacro (robot description, xacro)
@@ -50,16 +50,16 @@
                 <plugin>ign_ros2_control/IgnitionSystem</plugin>
             </hardware>
-            <xacro:wheel_transmission prefix="front" mechanical_reduction="20.0" can_network="can1"
-                motor_id="1" />
-            <xacro:wheel_transmission prefix="right" mechanical_reduction="20.0" can_network="can1"
-                motor_id="3" />
-            <xacro:wheel_transmission prefix="left" mechanical_reduction="20.0" can_network="can1"
-                motor_id="4" />
-            <xacro:wheel_transmission prefix="back" mechanical_reduction="20.0" can_network="can1"
-                motor_id="2" />
-            <xacro:gimbal_transmission prefix="yaw" mechanical_reduction="1.0" can_network="can1"
-                motor_id="5" />
-            <xacro:gimbal_transmission prefix="pitch" mechanical_reduction="-1.0" can_network="can1"
-                motor_id="6" />
+            <xacro:wheel_transmission prefix="front" mechanical_reduction="20.0" offset="0.0"
+                can_network="can1" motor_id="1" />
+            <xacro:wheel_transmission prefix="right" mechanical_reduction="20.0" offset="0.0"
+                can_network="can1" motor_id="3" />
+            <xacro:wheel_transmission prefix="left" mechanical_reduction="20.0" offset="0.0"
+                can_network="can1" motor_id="4" />
+            <xacro:wheel_transmission prefix="back" mechanical_reduction="20.0" offset="0.0"
+                can_network="can1" motor_id="2" />
+            <xacro:gimbal_transmission prefix="yaw" mechanical_reduction="1.0" offset="0.25"
+                can_network="can1" motor_id="5" />
+            <xacro:gimbal_transmission prefix="pitch" mechanical_reduction="-1.0" offset="0.0"
+                can_network="can1" motor_id="6" />
         </ros2_control>
     </xacro:if>
