Commit message: Add motor with external encoder to playground

File: decomposition/metav_description/urdf/playground/single_motor_ext_encoder.xacro (robot description, xacro)
@@ -1,4 +1,4 @@
 <?xml version="1.0"?>
-<robot name="multiple_motors" xmlns:xacro="http://www.ros.org/wiki/xacro">
+<robot name="single_motor" xmlns:xacro="http://www.ros.org/wiki/xacro">
     <xacro:arg name="is_simulation" default="true" />
     <link name="base_footprint">
@@ -12,6 +12,5 @@
     <link name="base_link" />
     <xacro:include filename="$(find metav_description)/urdf/playground/motor.xacro" />
-    <xacro:motor name="motor1" connected_to="base_link" x="0" y="0" />
-    <xacro:motor name="motor2" connected_to="base_link" x="3" y="0" />
+    <xacro:motor name="motor" connected_to="base_link" x="0" y="0" />
     <xacro:if value="$(arg is_simulation)">
         <ros2_control
@@ -20,15 +19,8 @@
                 <plugin>ign_ros2_control/IgnitionSystem</plugin>
             </hardware>
-            <joint name="motor1_joint">
-                <command_interface name="effort" />
+            <joint name="motor_joint">
+                <command_interface name="velocity" />
                 <state_interface name="position" />
                 <state_interface name="velocity" />
-                <state_interface name="effort" />
-            </joint>
-            <joint name="motor2_joint">
-                <command_interface name="position" />
-                <state_interface name="position" />
-                <state_interface name="velocity" />
-                <state_interface name="effort" />
             </joint>
         </ros2_control>
@@ -36,38 +28,34 @@
     <xacro:unless value="$(arg is_simulation)">
         <ros2_control
-            name="multiple_motors_control_dji" type="system">
-            <hardware>
-                <plugin>meta_hardware/MetaRobotDjiMotorNetwork</plugin>
-                <param name="can_network_name">can0</param>
-            </hardware>
-            <joint name="motor1_joint">
-                <command_interface name="effort" />
-                <state_interface name="position" />
-                <state_interface name="velocity" />
-                <state_interface name="effort" />
-                <param name="motor_model">GM6020</param>
-                <param name="motor_id">1</param>
-                <param name="mechanical_reduction">1.0</param>
-                <param name="offset">0.0</param>
-            </joint>
-        </ros2_control>
-        <ros2_control
-            name="multiple_motors_control_mi" type="system">
+            name="single_motor_control" type="system">
             <hardware>
                 <plugin>meta_hardware/MetaRobotMiMotorNetwork</plugin>
                 <param name="can_network_name">can0</param>
             </hardware>
-            <joint name="motor2_joint">
-                <command_interface name="position" />
-                <state_interface name="position" />
+            <joint name="motor_joint">
+                <command_interface name="velocity" />
                 <state_interface name="velocity" />
                 <state_interface name="effort" />
                 <param name="motor_model">CyberGear</param>
                 <param name="motor_id">1</param>
-                <param name="mechanical_reduction">1.0</param>
+                <param name="mechanical_reduction">-1.0</param>
                 <param name="offset">0.0</param>
                 <param name="control_mode">dynamic</param>
-                <param name="Kp">30.0</param>
+                <param name="Kp">0.0</param>
                 <param name="Kd">1.0</param>
+            </joint>
+        </ros2_control>
+        <ros2_control
+            name="single_motor_feedback" type="system">
+            <hardware>
+                <plugin>meta_hardware/MetaRobotBrtEncoderNetwork</plugin>
+                <param name="can_network_name">can0</param>
+            </hardware>
+            <joint name="motor_joint">
+                <state_interface name="position" />
+                <param name="encoder_model">BRT38-1024</param>
+                <param name="encoder_id">1</param>
+                <param name="mechanical_reduction">-1.0</param>
+                <param name="offset">0.0</param>
             </joint>
         </ros2_control>
@@ -78,5 +66,5 @@
             <plugin filename="ign_ros2_control-system"
                 name="ign_ros2_control::IgnitionROS2ControlPlugin">
-                <parameters>$(find meta_bringup)/config/multiple_motors.yaml</parameters>
+                <parameters>$(find meta_bringup)/config/single_motor_ext_encoder.yaml</parameters>
             </plugin>
         </gazebo>
