Commit message: shoot controller test

File: decomposition/metav_description/urdf/playground/shooter.xacro (robot description, xacro)
@@ -28,5 +28,5 @@
             </hardware>
         </xacro:unless>
-        <joint name="fric1_joint">
+        <joint name="friction_wheel1_joint">
             <command_interface name="effort" />
             <state_interface name="position" />
@@ -38,5 +38,5 @@
             <param name="offset">0.0</param>
         </joint>
-        <joint name="fric2_joint">
+        <joint name="friction_wheel2_joint">
             <command_interface name="effort" />
             <state_interface name="position" />
