Commit message: xacro modification

File: decomposition/metav_description/urdf/sentry25/sentry.chassis.xacro (robot description, xacro)
@@ -15,5 +15,5 @@
                 <origin xyz="0 0 0" rpy="0 0 0"/>
                 <geometry>
-                    <mesh filename="file://$(find metav_description)/meshes/sentry/chassis.stl" scale="1.0 1.0 1.0"/>
+                    <mesh filename="file://$(find metav_description)/meshes/sentry25/chassis.stl" scale="1.0 1.0 1.0"/>
                 </geometry>
                 <material name="silver">
@@ -28,20 +28,20 @@
             </collision>
         </link>
-        <xacro:omni_wheel prefix="front" connected_to="base_link"
+        <xacro:steer_wheel prefix="left_forward" connected_to="base_link"
                           wheel_x_offset="${chassis_radius}" wheel_y_offset="0.0"
                           wheel_z_offset="${wheel_offset_z}" rotation_degree="${-pi/2}" roller_type="${roller_type}"
                           max_effort="3.42" max_velocity="73"
         />
-        <xacro:omni_wheel prefix="right" connected_to="base_link"
+        <xacro:steer_wheel prefix="left_back" connected_to="base_link"
                           wheel_x_offset="0.0" wheel_y_offset="${-chassis_radius}"
                           wheel_z_offset="${wheel_offset_z}" rotation_degree="${pi}" roller_type="${roller_type}"
                           max_effort="3.42" max_velocity="73"
         />
-        <xacro:omni_wheel prefix="left" connected_to="base_link"
+        <xacro:steer_wheel prefix="right_forward" connected_to="base_link"
                           wheel_x_offset="0.0" wheel_y_offset="${chassis_radius}"
                           wheel_z_offset="${wheel_offset_z}" rotation_degree="${0}" roller_type="${roller_type}"
                           max_effort="3.42" max_velocity="73"
         />
-        <xacro:omni_wheel prefix="back" connected_to="base_link"
+        <xacro:steer_wheel prefix="right_back" connected_to="base_link"
                           wheel_x_offset="${-chassis_radius}" wheel_y_offset="${0}"
                           wheel_z_offset="${wheel_offset_z}" rotation_degree="${pi/2}" roller_type="${roller_type}"

File: decomposition/metav_description/urdf/sentry25/sentry.xacro (robot description, xacro)
@@ -33,8 +33,8 @@
                 <param name="can_network_name">can1</param>
             </hardware>
-            <xacro:wheel_transmission prefix="front" mechanical_reduction="20.0" motor_id="1" />
-            <xacro:wheel_transmission prefix="right" mechanical_reduction="20.0" motor_id="3" />
-            <xacro:wheel_transmission prefix="left" mechanical_reduction="20.0" motor_id="4" />
-            <xacro:wheel_transmission prefix="back" mechanical_reduction="20.0" motor_id="2" />
+            <xacro:wheel_transmission prefix="left_forward" mechanical_reduction="20.0" motor_id="1" />
+            <xacro:wheel_transmission prefix="left_back" mechanical_reduction="20.0" motor_id="3" />
+            <xacro:wheel_transmission prefix="right_forward" mechanical_reduction="20.0" motor_id="4" />
+            <xacro:wheel_transmission prefix="right_back" mechanical_reduction="20.0" motor_id="2" />
             <xacro:gimbal_transmission prefix="yaw" mechanical_reduction="1.0" offset="0.25"
                 motor_id="5" />
@@ -54,8 +54,8 @@
                 <plugin>ign_ros2_control/IgnitionSystem</plugin>
             </hardware>
-            <xacro:wheel_transmission prefix="front" mechanical_reduction="20.0" motor_id="1" />
-            <xacro:wheel_transmission prefix="right" mechanical_reduction="20.0" motor_id="3" />
-            <xacro:wheel_transmission prefix="left" mechanical_reduction="20.0" motor_id="4" />
-            <xacro:wheel_transmission prefix="back" mechanical_reduction="20.0" motor_id="2" />
+            <xacro:wheel_transmission prefix="left_forward" mechanical_reduction="20.0" motor_id="1" />
+            <xacro:wheel_transmission prefix="left_back" mechanical_reduction="20.0" motor_id="3" />
+            <xacro:wheel_transmission prefix="right_forward" mechanical_reduction="20.0" motor_id="4" />
+            <xacro:wheel_transmission prefix="right_back" mechanical_reduction="20.0" motor_id="2" />
             <xacro:gimbal_transmission prefix="yaw" mechanical_reduction="1.0" offset="0.25"
                 motor_id="5" />
