Commit message: agv chassis strange bug

File: decomposition/metav_description/urdf/common/steer_wheel.xacro (robot description, xacro)
@@ -58,5 +58,5 @@
         </joint>
     </xacro:macro>
-    <xacro:macro name="wheel_transmission" params="prefix mechanical_reduction motor_id">
+    <xacro:macro name="wheel_transmission" params="prefix mechanical_reduction vel_motor_id pos_motor_id pos_offset">
         <joint name="${prefix}_vel_joint">
             <command_interface name="effort">
@@ -66,5 +66,5 @@
             <state_interface name="effort" />
             <param name="motor_model">M3508</param>
-            <param name="motor_id">${motor_id}</param>
+            <param name="motor_id">${vel_motor_id}</param>
             <param name="mechanical_reduction">${mechanical_reduction}</param>
             <param name="offset">0.0</param>
@@ -77,7 +77,7 @@
             <state_interface name="effort" />
             <param name="motor_model">GM6020</param>
-            <param name="motor_id">${motor_id}</param>
-            <param name="mechanical_reduction">${mechanical_reduction}</param>
-            <param name="offset">0.0</param>
+            <param name="motor_id">${pos_motor_id}</param>
+            <param name="mechanical_reduction">1</param>
+            <param name="offset">${pos_offset}</param>
         </joint>
     </xacro:macro>

File: decomposition/metav_description/urdf/sentry25/sentry.xacro (robot description, xacro)
@@ -31,20 +31,20 @@
             <hardware>
                 <plugin>meta_hardware/MetaRobotDjiMotorNetwork</plugin>
-                <param name="can_network_name">can1</param>
+                <param name="can_network_name">can0</param>
             </hardware>
-            <xacro:wheel_transmission prefix="left_forward" mechanical_reduction="20.0" motor_id="1" />
-            <xacro:wheel_transmission prefix="left_back" mechanical_reduction="20.0" motor_id="3" />
-            <xacro:wheel_transmission prefix="right_forward" mechanical_reduction="20.0" motor_id="4" />
-            <xacro:wheel_transmission prefix="right_back" mechanical_reduction="20.0" motor_id="2" />
+            <xacro:wheel_transmission prefix="left_forward" mechanical_reduction="20.0" vel_motor_id="3" pos_motor_id="3" pos_offset="-0.0609"/>
+            <xacro:wheel_transmission prefix="left_back" mechanical_reduction="20.0" vel_motor_id="2" pos_motor_id = "1" pos_offset="0.1227"/>
+            <xacro:wheel_transmission prefix="right_forward" mechanical_reduction="20.0" vel_motor_id="4" pos_motor_id = "2" pos_offset="-0.0356"/>
+            <xacro:wheel_transmission prefix="right_back" mechanical_reduction="20.0" vel_motor_id="1" pos_motor_id = "4" pos_offset="-0.0694"/>
             <xacro:gimbal_transmission prefix="yaw" mechanical_reduction="1.0" offset="0.25"
                 motor_id="5" />
             <xacro:gimbal_transmission prefix="pitch" mechanical_reduction="-1.0" offset="0.0"
                 motor_id="6" />
-            <xacro:shooter_transmission prefix="fric1" mechanical_reduction="1.0" offset="0.25"
+            <!-- <xacro:shooter_transmission prefix="fric1" mechanical_reduction="1.0" offset="0.25"
                 motor_id="5" />
             <xacro:shooter_transmission prefix="fric2" mechanical_reduction="-1.0" offset="0.0"
                 motor_id="6" />
             <xacro:shooter_transmission prefix="loader" mechanical_reduction="36.0" offset="0.0"
-                motor_id="7" />
+                motor_id="7" /> -->
         </ros2_control>
     </xacro:unless>
