Commit message: fix motor interfaces

File: decomposition/metav_description/urdf/common/dm.xacro (robot description, xacro)
@@ -3,5 +3,5 @@
     <!-- motor_id should be in dec not hex otherwise it will not work -->
     <!-- mode: mit or posvelo(position-velocity mode) -->
-    <xacro:macro name="dm_motor" params="joint_name motor_id mode max_pos:=12.5 max_vel:=45.0 max_effort:=12.0 mechanical_reduction:=1.0 kp:=0.0 kd:=0.5">
+    <xacro:macro name="dm_motor" params="joint_name motor_id mode max_posvelo_vel:= 0.1 max_pos:=12.5 max_vel:=45.0 max_effort:=12.0 mechanical_reduction:=1.0 kp:=0.0 kd:=0.5">
         <joint name="${joint_name}">
                 <param name="control_mode">${mode}</param>
@@ -12,4 +12,8 @@
                 <param name="mechanical_reduction">${mechanical_reduction}</param>
                 <param name="offset">0.0</param>
+                <!-- below are the default values for the most motors, and please double check it before use-->
+                <param name="max_pos">${max_pos}</param>
+                <param name="max_vel">${max_vel}</param>
+                <param name="max_effort">${max_effort}</param>
                 <!-- mode dependent info-->
                 <xacro:if value="${mode == 'mit'}">
@@ -18,9 +22,5 @@
                     <command_interface name="effort"/>
                     <!-- max pos/vel/effort is written to dm motors(using the dm tool)-->
-                    <!-- below are the default values for the most motors, and please double check it before use-->
-                    <param name="max_pos">${max_pos}</param>
-                    <param name="max_vel">${max_vel}</param>
-                    <param name="max_effort">${max_effort}</param>
-                    <!-- kp kd only available in mit mode-->
+                    <!-- kp kd only available in mit mode, they are not property of motor but rather control signals sent to motors-->
                     <param name="kp">${kp}</param>
                     <param name="kd">${kd}</param>
@@ -30,5 +30,5 @@
                     <command_interface name="velocity"/>
                     <!-- if command of pos is valid and vel is nan, then use max_vel -->
-                    <param name="max_vel">${max_vel}</param>
+                    <param name="max_posvelo_vel">${max_posvelo_vel}</param>
                 </xacro:if>
                 <!-- state(feedback) are all available for all modes-->
