Commit message: fix hero xacro binding

File: decomposition/metav_description/urdf/hero/hero.xacro (robot description, xacro)
@@ -41,9 +41,45 @@
         <ros2_control name="dm_motors_yaw" type="system">
             <hardware>
-                <plugin>meta_hardware/MetaRobotDjiMotorNetwork</plugin>
+                <plugin>meta_hardware/MetaRobotDmMotorNetwork</plugin>
                 <param name="can_network_name">can_1</param>
+                <param name="master_id">0x30</param>
             </hardware>
-            <xacro:gimbal_transmission prefix="pitch" mechanical_reduction="20.0" motor_id="7" offset="0"/>
-            <xacro:gimbal_transmission prefix="yaw" mechanical_reduction="20.0" motor_id="8" offset="0"/>
+            <joint name="yaw_gimbal_joint">
+                <command_interface name="position" />
+                <state_interface name="position" />
+                <state_interface name="velocity" />
+                <state_interface name="effort" />
+                <param name="motor_model">DaMiao</param>
+                <param name="motor_id">9</param>
+                <param name="mechanical_reduction">1.0</param>
+                <param name="max_pos">12.5</param>
+                <param name="max_vel">45.0</param>
+                <param name="max_effort">12.0</param>
+                <param name="offset">0.0</param>
+                <param name="control_mode">mit</param>
+                <param name="Kp">30.0</param>
+                <param name="Kd">0.5</param>
+            </joint>
+        </ros2_control>
+        <ros2_control name="mi_motors_pitch" type="system">
+            <hardware>
+                <plugin>meta_hardware/MetaRobotMiMotorNetwork</plugin>
+                <param name="can_network_name">can_2</param>
+            </hardware>
+            <!-- <xacro:gimbal_transmission prefix="pitch" mechanical_reduction="20.0" motor_id="1" offset="0"/>
+             -->
+            <joint name="pitch_gimbal_joint">
+                <command_interface name="position" />
+                <state_interface name="position" />
+                <state_interface name="velocity" />
+                <state_interface name="effort" />
+                <param name="motor_model">CyberGear</param>
+                <param name="motor_id">1</param>
+                <param name="mechanical_reduction">1.0</param>
+                <param name="offset">0.7599</param> <!-- read from (int("7842",16)-65535/2)/(65535/2)*4*pi = -0.75990, remember to negate -->
+                <param name="control_mode">dynamic</param>
+                <param name="Kp">30.0</param>
+                <param name="Kd">1.0</param>
+            </joint>
         </ros2_control>
         <ros2_control name="dji_motors_gimbal" type="system">

File: decomposition/metav_description/urdf/playground/multiple_motors.xacro (robot description, xacro)
@@ -66,5 +66,7 @@
                 <param name="motor_id">1</param>
                 <param name="mechanical_reduction">1.0</param>
-                <param name="offset">0.0</param>
+                <!-- cansend can_2 01000001#0000.0000.0000.000 -->
+                <!-- can_2  020001FD   [8]  77 2C 7F F5 7F FF 01 2 -->
+                <param name="offset">0.86652061961</param> <!-- -0.7338292567 (int("772C",16)-65535/2)/(65535/2)*4*pi -->
                 <param name="control_mode">dynamic</param>
                 <param name="Kp">30.0</param>

Commit message: in jazzy ros2_control-only joints doesn't make sense, need to add dummy joints

File: decomposition/metav_description/urdf/hero/hero.xacro (robot description, xacro)
@@ -2,11 +2,37 @@
 <robot name="standard" xmlns:xacro="http://www.ros.org/wiki/xacro">
     <xacro:arg name="is_simulation" default="true" />
-    <link name="base_footprint">
-    </link>
     <!-- raise the robot a bit higher to prevent it from stucking in the ground -->
     <joint name="joint_base_to_footprint" type="fixed">
         <origin rpy="0 0 0" xyz="0 0 1" />
-        <parent link="base_footprint" />
+        <parent link="l0" />
         <child link="base_link" />
+    </joint>
+    <!-- dummy joints&links to suppress not found in URDF error-->
+    <link name="l0"/>
+    <link name="l1"/>
+    <link name="l2"/>
+    <link name="l3"/>
+    <link name="l4"/>
+    <link name="l5"/>
+    <!-- Fixed joints do not make sense in ros2_control-->
+    <joint name="loader_shooter_joint" type="continuous">
+        <parent link="l0" />
+        <child link="l1" />
+    </joint>
+    <joint name="yaw_gimbal_joint" type="continuous">
+        <parent link="l0" />
+        <child link="l2" />
+    </joint>
+    <joint name="pitch_gimbal_joint" type="continuous">
+        <parent link="l0" />
+        <child link="l3" />
+    </joint>
+    <joint name="fric1_shooter_joint" type="continuous">
+        <parent link="l0" />
+        <child link="l4" />
+    </joint>
+    <joint name="fric2_shooter_joint" type="continuous">
+        <parent link="l0" />
+        <child link="l5" />
     </joint>
     <xacro:include filename="$(find metav_description)/urdf/standard/standard.chassis.xacro" />

File: decomposition/metav_description/urdf/playground/cjh_chassis.xacro (robot description, xacro)
@@ -2,18 +2,37 @@
 <robot name="standard" xmlns:xacro="http://www.ros.org/wiki/xacro">
     <xacro:arg name="is_simulation" default="true" />
-    <link name="base_footprint">
-    </link>
-    <!-- raise the robot a bit higher to prevent it from stucking in the ground -->
-    <joint name="joint_base_to_footprint" type="fixed">
-        <origin rpy="0 0 0" xyz="0 0 1" />
-        <parent link="base_footprint" />
-        <child link="base_link" />
+    <!-- dummy joints&links to suppress not found in URDF error-->
+    <link name="l0"/>
+    <link name="l1"/>
+    <link name="l2"/>
+    <link name="l3"/>
+    <link name="l4"/>
+    <link name="l5"/>
+    <!-- Fixed joints do not make sense in ros2_control-->
+    <joint name="dummy_yaw_wheel_joint" type="continuous">
+        <parent link="l0" />
+        <child link="l1" />
+    </joint>
+    <joint name="front_left_wheel_joint" type="continuous">
+        <parent link="l0" />
+        <child link="l2" />
+    </joint>
+    <joint name="front_right_wheel_joint" type="continuous">
+        <parent link="l0" />
+        <child link="l3" />
+    </joint>
+    <joint name="back_left_wheel_joint" type="continuous">
+        <parent link="l0" />
+        <child link="l4" />
+    </joint>
+    <joint name="back_right_wheel_joint" type="continuous">
+        <parent link="l0" />
+        <child link="l5" />
     </joint>
     <xacro:include filename="$(find metav_description)/urdf/standard/standard.chassis.xacro" />
-    <xacro:chassis roller_type="none" />
     <ros2_control name="dji_motors_chassis" type="system">
         <hardware>
             <plugin>meta_hardware/MetaRobotDjiMotorNetwork</plugin>
-            <param name="can_network_name">can0</param>
+            <param name="can_network_name">can_1</param>
         </hardware>
         <xacro:wheel_transmission prefix="front_left" mechanical_reduction="20.0" motor_id="2" />
