Commit message: commit shit

File: decomposition/meta_manipulator/engineer_arm_moveit_config/config/engineer26.xacro (robot description, xacro)
@@ -1,12 +1,5 @@
 <?xml version="1.0"?>
-<robot name="standard" xmlns:xacro="http://www.ros.org/wiki/xacro">
-    <!-- dummy joints&links to suppress not found in URDF error-->
-    <joint name="joint_base_to_footprint" type="fixed">
-        <origin rpy="0 0 0" xyz="0 0 1" />
-        <parent link="l0" />
-        <child link="base_link" />
-    </joint>
-    <!-- dummy joints&links to suppress not found in URDF error-->
-    <link name="l0"/>
+<robot name="engineer26" xmlns:xacro="http://www.ros.org/wiki/xacro">
+    <xacro:include filename="$(find engineer_arm_moveit_config)/config/meta_arm.urdf.xacro" />
     <!-- TODO put that macro somewhere-->
     <xacro:macro name="shooter_transmission"
@@ -23,4 +16,5 @@
         </joint>
     </xacro:macro>
+    <!-- fix it-->
     <!-- note mecanum_wheel use dji motors-->
     <xacro:include filename="$(find metav_description)/urdf/common/mecanum_wheel.xacro"/>
@@ -28,5 +22,4 @@
     <xacro:include filename="$(find metav_description)/urdf/common/dm.xacro"/>
     <xacro:include filename="$(find metav_description)/urdf/standard/standard.chassis.xacro" />
-    <xacro:chassis roller_type="none" />
     <!-- chassis-->
     <ros2_control name="dji_motors_chassis" type="system">
@@ -79,5 +72,5 @@
             <param name="tty_devpath">/dev/ttyACM1</param>
         </hardware>
-        <xacro:unitree_go1_motor joint_name="joint3" motor_id="0" kp="1" kd="0.1" offset="1.368"/>
+        <xacro:unitree_go1_motor joint_name="joint3" motor_id="0" kp="1.5" kd="0.1" offset="-0.562"/>
     </ros2_control>
 </robot>

File: decomposition/meta_manipulator/engineer_arm_moveit_config/config/meta_arm.urdf.xacro (robot description, xacro)
@@ -5,5 +5,5 @@
     <xacro:include filename="$(find meta_arm_urdf)/urdf/meta_arm.urdf" />
     <!-- Import control_xacro -->
+    <!-- note: no need, since this file will be included by engineer26.xacro-->
     <xacro:include filename="meta_arm.ros2_control.xacro" />
-    <xacro:meta_arm_ros2_control name="FakeSystem" initial_positions_file="$(arg initial_positions_file)"/>
 </robot>

File: decomposition/meta_manipulator/meta_arm_urdf/urdf/meta_arm.urdf (robot description, URDF)
Before this commit: robot meta_arm, 8 links, 7 joints
Links:
- added link gunmu1
- added link gunmu2
- added link gunmu3
- added link gunmu4
- added link gunmu5
- added link gunmu6
Joints:
- added joint back_left_wheel_joint: type revolute, parent base, child gunmu2, axis -1 0 0, limit lower=-3.14 upper=3.14 effort=0 velocity=1.0
- added joint back_right_wheel_joint: type revolute, parent base, child gunmu5, axis -1 0 0, limit lower=-3.14 upper=3.14 effort=0 velocity=1.0
- added joint dummy_yaw_wheel_joint: type revolute, parent base, child gunmu6, axis -1 0 0, limit lower=-3.14 upper=3.14 effort=0 velocity=1.0
- added joint front_left_wheel_joint: type revolute, parent base, child gunmu3, axis -1 0 0, limit lower=-3.14 upper=3.14 effort=0 velocity=1.0
- added joint front_right_wheel_joint: type revolute, parent base, child gunmu4, axis -1 0 0, limit lower=-3.14 upper=3.14 effort=0 velocity=1.0
- added joint joint_end_eff_shooter_joint: type revolute, parent base, child gunmu1, axis -1 0 0, limit lower=-3.14 upper=3.14 effort=0 velocity=1.0
- joint joint3: limit lower=-1.57 upper=1.57 effort=0 velocity=1.0 -> lower=-1.57 upper=2.5 effort=0 velocity=1.0
